File: flash.kicad_sch (KiCad schematic)
At the start: 2 parts, among them U3 W25Q128JVS

Commit message: fix(pcb): populate footprints for C1..C24, R1..R14, J1, J3, L1, L2, Y1 across all schematic sheets to eliminate import errors
Parts:
- C20: footprint (none) -> Capacitor_SMD:C_0805_2012Metric
Changed lines of the file:
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@@
 			)
 		)
-		(property "Footprint" ""
+		(property "Footprint" "Capacitor_SMD:C_0805_2012Metric"
 			(at 135.89 54.9148 0)
 			(effects

Commit message: Update passive component footprints to 0603 and sync DRC rules
Parts:
- C20: footprint Capacitor_SMD:C_0805_2012Metric -> Capacitor_SMD:C_0603_1608Metric
Changed lines of the file:
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@@
 			)
 		)
-		(property "Footprint" "Capacitor_SMD:C_0805_2012Metric"
+		(property "Footprint" "Capacitor_SMD:C_0603_1608Metric"
 			(at 135.89 54.9148 0)
 			(effects
