File: flash.kicad_sch (KiCad schematic)
At the start: 2 parts, among them U3 W25Q128JVS

Commit message: Complete schematic for first prototype
- Footprints: passives 0402/0603 (larger only for 24 V / DC bias),
  U1 and L1 footprints taken from RP2350A Minimal R4 reference (MIT)
- New sheet vystupy: heater (Q1 SiS434DN) with thermal fuse terminal J13,
  fan (GPIO13) and exhaust fan (GPIO12) with AO3422, input protection
  (fuse, AOD4185 reverse polarity, SMBJ24CA TVS, bulk cap), status LED on
  RM2 GPIO0, button GPIO15, NTC on ADC0 (22k pull-up), I2C1 pull-ups,
  second SHT40 on I2C0 (GPIO8/9)
- New sheet rozsireni: spare GPIO header J12, test points TP1-TP5,
  mounting holes H1-H4
- Selected parts with Manufacturer/MPN fields; L2 4.7 uH Wurth 74438356047
- Fix D2 pin mapping (Device:D_Schottky), remove duplicate pull-down R12,
  C16 changed to 100 nF for third DVDD pin, Y1 value set
- Project footprint library susicka.pretty (PowerPAK 1212-8 with G/S/D pads)

Co-Authored-By: Claude Opus 5.5 <noreply@anthropic.com>
Parts:
- C20: footprint Capacitor_SMD:C_0603_1608Metric -> Capacitor_SMD:C_0402_1005Metric
Changed lines of the file:
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@@
 			)
 		)
-		(property "Footprint" "Capacitor_SMD:C_0603_1608Metric"
+		(property "Footprint" "Capacitor_SMD:C_0402_1005Metric"
 			(at 135.89 54.9148 0)
 			(effects
