File: pwr.kicad_sch (KiCad schematic)
At the start: 7 parts, among them J4 PJ-102AH, U4 AP63203WU

Commit message: Replace Gemini-generated layout with clean project for manual layout
Remove generated scripts, test boards, DRC reports, renders and build
output; restore the sandbox project so the PCB layout can be done by hand.

Co-Authored-By: Claude Opus 5.5 <noreply@anthropic.com>
Parts:
- C21, C23, C24: footprint Capacitor_SMD:C_0805_2012Metric -> Capacitor_SMD:C_0603_1608Metric
Changed lines of the file:
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@@
 			)
 		)
-		(property "Footprint" "Capacitor_SMD:C_0805_2012Metric"
+		(property "Footprint" "Capacitor_SMD:C_0603_1608Metric"
 			(at 166.0652 102.87 0)
 			(effects
@@
 			)
 		)
-		(property "Footprint" "Capacitor_SMD:C_0805_2012Metric"
+		(property "Footprint" "Capacitor_SMD:C_0603_1608Metric"
 			(at 228.2952 101.6 0)
 			(effects
@@
 			)
 		)
-		(property "Footprint" "Capacitor_SMD:C_0805_2012Metric"
+		(property "Footprint" "Capacitor_SMD:C_0603_1608Metric"
 			(at 223.2152 101.6 0)
 			(effects

Commit message: Complete schematic for first prototype
- Footprints: passives 0402/0603 (larger only for 24 V / DC bias),
  U1 and L1 footprints taken from RP2350A Minimal R4 reference (MIT)
- New sheet vystupy: heater (Q1 SiS434DN) with thermal fuse terminal J13,
  fan (GPIO13) and exhaust fan (GPIO12) with AO3422, input protection
  (fuse, AOD4185 reverse polarity, SMBJ24CA TVS, bulk cap), status LED on
  RM2 GPIO0, button GPIO15, NTC on ADC0 (22k pull-up), I2C1 pull-ups,
  second SHT40 on I2C0 (GPIO8/9)
- New sheet rozsireni: spare GPIO header J12, test points TP1-TP5,
  mounting holes H1-H4
- Selected parts with Manufacturer/MPN fields; L2 4.7 uH Wurth 74438356047
- Fix D2 pin mapping (Device:D_Schottky), remove duplicate pull-down R12,
  C16 changed to 100 nF for third DVDD pin, Y1 value set
- Project footprint library susicka.pretty (PowerPAK 1212-8 with G/S/D pads)

Co-Authored-By: Claude Opus 5.5 <noreply@anthropic.com>
Parts:
- C21: footprint Capacitor_SMD:C_0603_1608Metric -> Capacitor_SMD:C_1210_3225Metric
- C23, C24: footprint Capacitor_SMD:C_0603_1608Metric -> Capacitor_SMD:C_0805_2012Metric
- L2: value 3,9 uH -> 4,7uH; footprint Inductor_SMD:L_0805_2012Metric -> Inductor_SMD:L_Wuerth_MAPI-4020; MPN (none) -> 74438356047; Manufacturer (none) -> Würth Elektronik
Connections:
- net 24V: no longer J4.1
- new net 24V_IN: J4.1
Changed lines of the file:
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@@
 		)
 	)
-	(global_label "24V"
+	(global_label "24V_IN"
 		(shape output)
 		(at 140.97 85.09 0)
@@
 			)
 		)
-		(property "Value" "3,9 uH"
+		(property "Value" "4,7uH"
 			(at 210.82 73.66 90)
 			(effects
@@
 			)
 		)
-		(property "Footprint" "Inductor_SMD:L_0805_2012Metric"
+		(property "Footprint" "Inductor_SMD:L_Wuerth_MAPI-4020"
 			(at 210.82 76.2 0)
 			(effects
@@
 			)
 		)
-		(property "Description" "Inductor"
+		(property "Description" "WE-MAPI 4020, 4,7 uH, Irated 2,9 A, DCR 76 mOhm – cívka AP63203 (datasheet 3,9 uH; 4,7 uH jako SparkFun BabyBuck)"
+			(at 210.82 76.2 0)
+			(effects
+				(font
+					(size 1.27 1.27)
+				)
+				(hide yes)
+			)
+		)
+		(property "Manufacturer" "Würth Elektronik"
+			(at 210.82 76.2 0)
+			(effects
+				(font
+					(size 1.27 1.27)
+				)
+				(hide yes)
+			)
+		)
+		(property "MPN" "74438356047"
 			(at 210.82 76.2 0)
 			(effects
@@
 			)
 		)
-		(property "Footprint" "Capacitor_SMD:C_0603_1608Metric"
+		(property "Footprint" "Capacitor_SMD:C_1210_3225Metric"
 			(at 166.0652 102.87 0)
 			(effects
@@
 			)
 		)
-		(property "Footprint" "Capacitor_SMD:C_0603_1608Metric"
+		(property "Footprint" "Capacitor_SMD:C_0805_2012Metric"
 			(at 228.2952 101.6 0)
 			(effects
@@
 			)
 		)
-		(property "Footprint" "Capacitor_SMD:C_0603_1608Metric"
+		(property "Footprint" "Capacitor_SMD:C_0805_2012Metric"
 			(at 223.2152 101.6 0)
 			(effects
